Commit message: Release v2.0.0: 灵巧手挂载、视觉追踪优化与方向修正
- 新增 Allegro Hand 16关节灵巧手，连接至 RM65 末端 Link6
  (PAL Robotics, Apache-2.0)，手腕偏移 7cm 正位挂载
- 新增身体方向检测：基于肩膀线斜率 + 鼻耳偏移
  正对镜头时自动收紧 J1 锁定阈值(0.05→0.15)
- UI 面板实时显示身体角、水平模，正对时红色警告+侧身提示
- J1 左右方向修正 scale 1.0 (原 -1.0)，手左移→臂左移
- 新增 sim_hand_bridge / sim_hand_client 仿真灵巧手控制
- Gazebo 手势演示场景：RM65 + Allegro + 桌面 + ArUco 标记
- README 补充灵巧手部署说明与调参指南

Co-authored-by: Cursor <cursoragent@cursor.com>

File: vendor/ros2_rm_robot/rm_gazebo/config/gazebo_65_gesture.urdf.xacro (robot description, xacro)
@@ -1,4 +1,6 @@
 <?xml version="1.0"?>
 <robot xmlns:xacro="http://www.ros.org/wiki/xacro" name="rm_65_description">
+    <xacro:arg name="use_sim_time" default="true"/>
+    <xacro:arg name="pid_controllers" default="false"/>
     <link name="world"/>
     <joint name="fixed" type="fixed">
@@ -7,4 +9,13 @@
     </joint>
     <xacro:include filename="$(find rm_description)/urdf/rm_65_gazebo.urdf" />
+    <xacro:include filename="$(find allegro_hand_description)/urdf/allegro_hand.urdf.xacro" />
+    <xacro:include filename="$(find allegro_hand_description)/urdf/allegro_hand.ros2_control.xacro" />
+    <!-- Allegro Hand (PAL Robotics, Apache-2.0) -->
+    <!-- palm_link origin (hand root) mates to Link6 flange face -->
+    <!-- xyz: 7cm wrist offset along Link6 Z (arm axis direction) -->
+    <!-- rpy: 0 0 0 — no rotation, palm Z = Link6 Z = arm axis, fingers extend along arm direction -->
+    <xacro:allegro_hand name="gripper" parent="Link6" reflect="1">
+        <origin xyz="0.0 0.0 0.07" rpy="0 0 0"/>
+    </xacro:allegro_hand>
     <link name="arm_camera_link">
         <visual>
@@ -60,4 +71,8 @@
     <gazebo reference="link6">
         <material>Gazebo/Orange</material>
+        <gravity>false</gravity>
+    </gazebo>
+    <gazebo reference="gripper_palm_link">
+        <material>Gazebo/DarkGrey</material>
         <gravity>false</gravity>
     </gazebo>
@@ -142,4 +157,5 @@
             <state_interface name="velocity"/>
         </joint>
+        <xacro:ros2_control_allegro_hand name="gripper" pid_controllers="$(arg pid_controllers)" reduction="1.0"/>
     </ros2_control>
     <gazebo>
